Commit message: fixed t_block

File: assets/t_block.urdf (robot description, URDF)
Before this commit: robot t_block, 1 links, 0 joints
Links:
- added link p1
- added link p2
- added link p3
- added link p4
- added link p5
- added link p6
- added link p7
- added link p8
- link t_block: mass 0.225 -> 0.60; geometry collision box size=0.05 0.20 0.05; collision box size=0.20 0.05 0.05
Joints:
- added joint t_block_p1: type fixed, parent t_block, child p1, origin xyz=-0.025 -0.125 0 rpy=0 0 0
- added joint t_block_p2: type fixed, parent t_block, child p2, origin xyz=-0.025 0.075 0 rpy=0 0 0
- added joint t_block_p3: type fixed, parent t_block, child p3, origin xyz=-0.10 0.075 0 rpy=0 0 0
- added joint t_block_p4: type fixed, parent t_block, child p4, origin xyz=-0.10 0.125 0 rpy=0 0 0
- added joint t_block_p5: type fixed, parent t_block, child p5, origin xyz=0.10 0.125 0 rpy=0 0 0
- added joint t_block_p6: type fixed, parent t_block, child p6, origin xyz=0.10 0.075 0 rpy=0 0 0
- added joint t_block_p7: type fixed, parent t_block, child p7, origin xyz=0.025 0.075 0 rpy=0 0 0
- added joint t_block_p8: type fixed, parent t_block, child p8, origin xyz=0.025 -0.125 0 rpy=0 0 0
